Commit message: Update panda_arm_hand.srdf.xacro
see franka_ros version 0.7.1

File: config/panda_arm_hand.srdf.xacro (robot description, xacro)
@@ -18,26 +18,29 @@
     <group name="hand" />
   </group>
-  <group_state name="open" group="hand">
-    <joint name="panda_finger_joint1" value="0.035" />
-    <joint name="panda_finger_joint2" value="0.035" />
-  </group_state>
-  <group_state name="close" group="hand">
-    <joint name="panda_finger_joint1" value="0" />
-    <joint name="panda_finger_joint2" value="0" />
+  <!--GROUP STATES: Purpose: Define a named state for a particular group, in terms of joint values. This is useful to define states like 'folded arms'-->
+  <group_state name="ready" group="panda_arm_hand">
+    <joint name="panda_joint1" value="0" />
+    <joint name="panda_joint2" value="-0.785" />
+    <joint name="panda_joint3" value="0" />
+    <joint name="panda_joint4" value="-2.356" />
+    <joint name="panda_joint5" value="0" />
+    <joint name="panda_joint6" value="1.571" />
+    <joint name="panda_joint7" value="0.785" />
   </group_state>
   <!--END EFFECTOR: Purpose: Represent information about an end effector.-->
-  <end_effector name="hand" parent_link="panda_link8" group="hand" parent_group="panda_arm" />
+  <end_effector name="hand" parent_link="panda_hand" group="hand" parent_group="panda_arm_hand" />
   <!--DISABLE COLLISIONS: By default it is assumed that any link of the robot could potentially come into collision with any other link in the robot. This tag disables collision checking between a specified pair of links. -->
+  <disable_collisions link1="panda_hand" link2="panda_link3" reason="Never" />
   <disable_collisions link1="panda_hand" link2="panda_link4" reason="Never" />
+  <disable_collisions link1="panda_hand" link2="panda_link5" reason="Default" />
   <disable_collisions link1="panda_hand" link2="panda_link6" reason="Never" />
-  <disable_collisions link1="panda_hand" link2="panda_link7" reason="Default" />
-  <disable_collisions link1="panda_hand" link2="panda_link8" reason="Adjacent" />
+  <disable_collisions link1="panda_hand" link2="panda_link7" reason="Adjacent" />
+  <disable_collisions link1="panda_leftfinger" link2="panda_link3" reason="Never" />
   <disable_collisions link1="panda_leftfinger" link2="panda_link4" reason="Never" />
   <disable_collisions link1="panda_leftfinger" link2="panda_link6" reason="Never" />
   <disable_collisions link1="panda_leftfinger" link2="panda_link7" reason="Never" />
-  <disable_collisions link1="panda_leftfinger" link2="panda_link8" reason="Never" />
+  <disable_collisions link1="panda_link3" link2="panda_rightfinger" reason="Never" />
   <disable_collisions link1="panda_link4" link2="panda_rightfinger" reason="Never" />
   <disable_collisions link1="panda_link6" link2="panda_rightfinger" reason="Never" />
   <disable_collisions link1="panda_link7" link2="panda_rightfinger" reason="Never" />
-  <disable_collisions link1="panda_link8" link2="panda_rightfinger" reason="Never" />
 </robot>
